Commit message: added camera functionality

File: src/double_inverted_pendulum/description/pendulum2.urdf.xacro (robot description, xacro)
@@ -12,4 +12,5 @@
     <xacro:property name="pendulumdamping" value="0.0" />
     <xacro:property name="pendulumfriction" value="0.10" />
+    <xacro:property name="camerasize" value="0.10" />
     <!-- #endregion -->
     <!-- #region MAKE_BOX -->
@@ -75,10 +76,10 @@
     <!-- #region BASE -->
     <link name="base_link">
-        <xacro:make_box length="0.5" width="0.5" height="${boxheight}" mass="1000" material="red" originxyz="0 0 0" originrpy="0 0 0"/>
+        <xacro:make_box length="0.5" width="0.5" height="${boxheight}" mass="10" material="red" originxyz="0 0 0" originrpy="0 0 0"/>
     </link>
     <!-- #endregion -->
     <!-- #region PENDULUM_JOINT -->
     <link name="pendulum_joint">
-        <xacro:make_box length="${pendulumwidth}" width="${pendulumwidth}" height="${pendulumwidth*2}" mass="10" material="red" originxyz="0 0 ${-pendulumwidth/2}" originrpy="0 0 0"/>
+        <xacro:make_box length="${pendulumwidth}" width="${pendulumwidth}" height="${pendulumwidth*2}" mass="100" material="red" originxyz="0 0 ${-pendulumwidth/2}" originrpy="0 0 0"/>
     </link>
     <joint name="base_to_pendulum_joint" type="fixed">
@@ -91,5 +92,5 @@
     <!-- #region FIRST_PENDULUM -->
     <link name="first_pendulum">
-        <xacro:make_box length="${pendulumwidth}" width="${pendulumwidth}" height="${pendulumlength}" mass="2" material="black" originxyz="0 0 ${pendulumlength/2 - pendulumwidth/2}" originrpy="0 0 0"/>
+        <xacro:make_box length="${pendulumwidth}" width="${pendulumwidth}" height="${pendulumlength}" mass="10" material="black" originxyz="0 0 ${pendulumlength/2 - pendulumwidth/2}" originrpy="0 0 0"/>
     </link>
     <joint name="pendulum_joint_to_first_pendulum" type="continuous">
@@ -104,5 +105,5 @@
     <!-- #region SECOND_PENDULUM -->
     <link name="second_pendulum">
-        <xacro:make_box length="${pendulumwidth}" width="${pendulumwidth}" height="${pendulumlength}" mass="2" material="red" originxyz="0 0 ${pendulumlength/2 - pendulumwidth/2}" originrpy="0 0 0"/>
+        <xacro:make_box length="${pendulumwidth}" width="${pendulumwidth}" height="${pendulumlength}" mass="10" material="red" originxyz="0 0 ${pendulumlength/2 - pendulumwidth/2}" originrpy="0 0 0"/>
     </link>
     <joint name="first_pendulum_to_second_pendulum" type="continuous">
@@ -118,5 +119,5 @@
     <!-- #region FRONT_LEFT_WHEEL -->
     <link name="front_left_wheel">
-        <xacro:make_cylinder length="0.1" radius="0.1" mass="0.3" material="orange" originxyz="0.051 0 0" originrpy="0 1.570796327 0"/>
+        <xacro:make_cylinder length="0.1" radius="0.1" mass="5" material="orange" originxyz="0.051 0 0" originrpy="0 1.570796327 0"/>
     </link>
     <joint name="base_to_front_left_wheel" type="continuous">
@@ -127,18 +128,8 @@
         <axis xyz="1 0 0"/>
     </joint>
-    <transmission name="FLWheel">
-        <type>transmission_interface/SimpleTransmission</type>
-        <joint name="base_to_front_left_wheel">
-            <hardwareInterface>hardware_interface/EffortJointInterface</hardwareInterface>
-        </joint>
-        <actuator name="FLWheel">
-            <hardwareInterface>hardware_interface/EffortJointInterface</hardwareInterface>
-            <mechanicalReduction>1</mechanicalReduction>
-        </actuator>
-    </transmission>
     <!-- #endregion -->
     <!-- #region FRONT_RIGHT_WHEEL -->
     <link name="front_right_wheel">
-        <xacro:make_cylinder length="0.1" radius="0.1" mass="0.3" material="orange" originxyz="0.051 0 0" originrpy="0 -1.570796327 0"/>
+        <xacro:make_cylinder length="0.1" radius="0.1" mass="5" material="orange" originxyz="0.051 0 0" originrpy="0 -1.570796327 0"/>
     </link>
     <joint name="base_to_front_right_wheel" type="continuous">
@@ -149,18 +140,8 @@
         <axis xyz="1 0 0"/>
     </joint>
-    <transmission name="FRWheel">
-        <type>transmission_interface/SimpleTransmission</type>
-        <joint name="base_to_front_right_wheel">
-            <hardwareInterface>hardware_interface/EffortJointInterface</hardwareInterface>
-        </joint>
-        <actuator name="FRWheel">
-            <hardwareInterface>hardware_interface/EffortJointInterface</hardwareInterface>
-            <mechanicalReduction>1</mechanicalReduction>
-        </actuator>
-    </transmission>
     <!-- #endregion -->
     <!-- #region BACK_LEFT_WHEEL -->
     <link name="back_left_wheel">
-        <xacro:make_cylinder length="0.1" radius="0.1" mass="0.3" material="orange" originxyz="-0.051 0 0" originrpy="0 1.570796327 0"/>
+        <xacro:make_cylinder length="0.1" radius="0.1" mass="5" material="orange" originxyz="-0.051 0 0" originrpy="0 1.570796327 0"/>
     </link>
     <joint name="base_to_back_left_wheel" type="continuous">
@@ -171,18 +152,8 @@
         <axis xyz="1 0 0"/>
     </joint>
-    <transmission name="BLWheel">
-        <type>transmission_interface/SimpleTransmission</type>
-        <joint name="base_to_back_left_wheel">
-            <hardwareInterface>hardware_interface/EffortJointInterface</hardwareInterface>
-        </joint>
-        <actuator name="BLWheel">
-            <hardwareInterface>hardware_interface/EffortJointInterface</hardwareInterface>
-            <mechanicalReduction>1</mechanicalReduction>
-        </actuator>
-    </transmission>
     <!-- #endregion -->
     <!-- #region BACK_RIGHT_WHEEL -->
     <link name="back_right_wheel">
-        <xacro:make_cylinder length="0.1" radius="0.1" mass="0.3" material="orange" originxyz="-0.051 0 0" originrpy="0 1.570796327 0"/>
+        <xacro:make_cylinder length="0.1" radius="0.1" mass="5" material="orange" originxyz="-0.051 0 0" originrpy="0 1.570796327 0"/>
     </link>
     <joint name="base_to_back_right_wheel" type="continuous">
@@ -193,15 +164,16 @@
         <axis xyz="1 0 0"/>
     </joint>
-    <transmission name="BRWheel">
-        <type>transmission_interface/SimpleTransmission</type>
-        <joint name="base_to_back_right_wheel">
-            <hardwareInterface>hardware_interface/EffortJointInterface</hardwareInterface>
-        </joint>
-        <actuator name="BRWheel">
-            <hardwareInterface>hardware_interface/EffortJointInterface</hardwareInterface>
-            <mechanicalReduction>1</mechanicalReduction>
-        </actuator>
-    </transmission>
     <!-- #endregion -->
     <!-- #endregion -->
+    <!-- #region CAMERA -->
+    <link name="camera">
+        <xacro:make_box length="${camerasize}" width="${camerasize}" height="${camerasize}" mass="1" material="white" originxyz="0 0 ${camerasize/2}" originrpy="0 0 0"/>
+    </link>
+    <joint name="base_to_camera" type="fixed">
+        <axis xyz="0 1 0" />
+        <origin xyz="0 ${0.5/2} ${boxheight/2}" rpy="0 0 1.57"/>
+        <parent link="base_link"/>
+        <child link="camera"/>
+    </joint>
+    <!-- #endregion -->
 </robot>

Commit message: added actor critic, fingers crossed

File: src/double_inverted_pendulum/description/pendulum2.urdf.xacro (robot description, xacro)
@@ -11,5 +11,5 @@
     <xacro:property name="pitchlimit" value="0" />
     <xacro:property name="pendulumdamping" value="0.0" />
-    <xacro:property name="pendulumfriction" value="0.10" />
+    <xacro:property name="pendulumfriction" value="0.30" />
     <xacro:property name="camerasize" value="0.10" />
     <!-- #endregion -->

Commit message: minor update to reward function

File: src/double_inverted_pendulum/description/pendulum2.urdf.xacro (robot description, xacro)
@@ -11,5 +11,5 @@
     <xacro:property name="pitchlimit" value="0" />
     <xacro:property name="pendulumdamping" value="0.0" />
-    <xacro:property name="pendulumfriction" value="0.30" />
+    <xacro:property name="pendulumfriction" value="0.50" />
     <xacro:property name="camerasize" value="0.10" />
     <!-- #endregion -->
@@ -113,5 +113,5 @@
         <origin xyz="${-pendulumwidth - 0.003} 0 ${pendulumlength - pendulumwidth}"/>
         <axis xyz="1 0 0"/>
-        <dynamics friction="${pendulumfriction}" damping="${pendulumdamping}"/>
+        <dynamics friction="1000" damping="${pendulumdamping}"/>
     </joint>
     <!-- #endregion -->

Commit message: add critic component of actor critic, not working

File: src/double_inverted_pendulum/description/pendulum2.urdf.xacro (robot description, xacro)
@@ -6,5 +6,5 @@
     <!-- #region CONSTANTS -->
     <xacro:property name="boxheight" value="0.1" />
-    <xacro:property name="pendulumlength" value="0.5" />
+    <xacro:property name="pendulumlength" value="0.75" />
     <xacro:property name="pendulummass" value="1" />
     <xacro:property name="pendulumwidth" value="0.05" />

Commit message: DOUBLE INVERTED PENDULUM

File: src/double_inverted_pendulum/description/pendulum2.urdf.xacro (robot description, xacro)
@@ -11,5 +11,5 @@
     <xacro:property name="pitchlimit" value="0" />
     <xacro:property name="pendulumdamping" value="0.0" />
-    <xacro:property name="pendulumfriction" value="0.50" />
+    <xacro:property name="pendulumfriction" value="0.01" />
     <xacro:property name="camerasize" value="0.10" />
     <!-- #endregion -->
@@ -113,5 +113,5 @@
         <origin xyz="${-pendulumwidth - 0.003} 0 ${pendulumlength - pendulumwidth}"/>
         <axis xyz="1 0 0"/>
-        <dynamics friction="1000" damping="${pendulumdamping}"/>
+        <dynamics friction="${pendulumfriction}" damping="${pendulumdamping}"/>
     </joint>
     <!-- #endregion -->
